File: Hardware/LuminX PWM.kicad_pcb (KiCad board)
At the start: 4 copper layers, 94.6 x 64.6 mm, 110 parts, among them J1 USB_C_Receptacle_USB2.0, J2 5mm Screw Terminal, J3 USB_B_Micro, J4 Conn_01x04_Pin, J5 Barrel_Jack_Switch, J6 Screw_Terminal_01x03, J7 5mm Screw Terminal, J9 Conn_01x03_Pin, Q1 BC847, Q10 BC847, Q11 BC847, Q12 BC847, Q13 BC847, Q2 BC847, Q3 BC847, Q4 IRLR8726, Q5 WSF70P03, Q6 IRLR8726, Q7 IRLR8726, Q8 IRLR8726, Q9 IRLR8726, SW2 SW_Push, SW3 SW_Push, U1 CH340G, U2 USBLC6-2P6, U3 ESP32-WROOM-32D, U4 TSOP382xx, U5 TPS54332, U6 AP2112K-3.3, U7 DS18B20, U8 INA180A1, Y1 12MHz

Commit message: update readme
Parts:
- renumbered H2 to He
Changed lines of the file:
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@@
     (property "ki_description" "Mounting Hole with connection")
     (property "ki_keywords" "mounting hole")
-    (attr exclude_from_pos_files)
+    (attr exclude_from_pos_files exclude_from_bom)
     (fp_text reference "H4" (at 0 -4.2) (layer "F.SilkS") hide
         (effects (font (size 1 1) (thickness 0.15)))
@@
     (property "ki_description" "Mounting Hole with connection")
     (property "ki_keywords" "mounting hole")
-    (attr exclude_from_pos_files)
+    (attr exclude_from_pos_files exclude_from_bom)
     (fp_text reference "H1" (at 0 -4.2) (layer "F.SilkS") hide
         (effects (font (size 1 1) (thickness 0.15)))
@@
     (property "ki_description" "Mounting Hole with connection")
     (property "ki_keywords" "mounting hole")
-    (attr exclude_from_pos_files)
-    (fp_text reference "H2" (at 0 -4.2) (layer "F.SilkS") hide
+    (attr exclude_from_pos_files exclude_from_bom)
+    (fp_text reference "He" (at 0 -4.2) (layer "F.SilkS") hide
         (effects (font (size 1 1) (thickness 0.15)))
     )
@@
     (property "ki_description" "Mounting Hole with connection")
     (property "ki_keywords" "mounting hole")
-    (attr exclude_from_pos_files)
+    (attr exclude_from_pos_files exclude_from_bom)
     (fp_text reference "H3" (at 0 -4.2) (layer "F.SilkS") hide
         (effects (font (size 1 1) (thickness 0.15)))
