File: Hardware/LuminX PWM.kicad_pcb (KiCad board)
At the start: 4 copper layers, 94.6 x 64.6 mm, 92 parts, among them J1 USB_C_Receptacle_USB2.0, J2 5mm Screw Terminal, J3 Barrel_Jack_Switch, J4 Conn_01x04_Pin, J5 5mm Screw Terminal, J9 Conn_01x03_Pin, Q1 BC847, Q10 BC847, Q11 BC847, Q12 BC847, Q13 BC847, Q14 AO3401A, Q2 BC847, Q3 BC847, Q4 IRLR8726, Q5 AOD4185, Q6 IRLR8726, Q7 IRLR8726, Q8 IRLR8726, Q9 IRLR8726, SW2 SW_Push, SW3 SW_Push, U1 CH340G, U2 USBLC6-2P6, U3 ESP32-WROOM-32D, U4 TSOP382xx, U5 AP62300WU, U6 AP2112K-3.3, U7 DS18B20, U8 LM321, Y1 12MHz

Commit message: Update backups
Parts:
- removed J9: Conn_01x03_Pin, Connector_PinHeader_2.54mm:PinHeader_1x03_P2.54mm_Vertical
- removed U5: AP62300WU, Package_TO_SOT_SMD:TSOT-23-6
- removed U8: LM321, Package_TO_SOT_SMD:SOT-23-5
- removed Y1: 12MHz, Crystal:Crystal_SMD_3225-4Pin_3.2x2.5mm
- added C17: 10u, Capacitor_SMD:C_1206_3216Metric, F.Cu at (106.0, 147.8)
- added D2: SS34, Diode_SMD:D_SMA, F.Cu at (107.3, 143.8)
- added R35: 10k, Resistor_SMD:R_0805_2012Metric, F.Cu at (111.1, 147.6)
- added U9: CH340C, Package_SO:SOIC-16_3.9x9.9mm_P1.27mm, F.Cu at (107.4, 157.4)
- C11, C15: footprint Capacitor_SMD:C_0805_2012Metric -> Capacitor_SMD:C_1206_3216Metric
- C5: value 30p -> 10n
- C7: footprint Capacitor_SMD:C_0603_1608Metric -> Capacitor_SMD:C_1206_3216Metric
- C8: value 10u -> 100n; footprint Diode_SMD:D_0805_2012Metric -> Capacitor_SMD:C_0603_1608Metric
- FB1: value 100R -> 100R 3A
- U1: value CH340G -> ESP32-WROOM-32E; footprint Package_SO:SOIC-16_3.9x9.9mm_P1.27mm -> RF_Module:ESP32-WROOM-32D
- U2: value USBLC6-2P6 -> AP63200WU; footprint Package_TO_SOT_SMD:SOT-666 -> Package_TO_SOT_SMD:TSOT-23-6
- U3: value ESP32-WROOM-32D -> USBLC6-2SC6; footprint RF_Module:ESP32-WROOM-32D -> Package_TO_SOT_SMD:SOT-23-6
- moved U2 35.9 mm to (127.2, 117.2)
- moved R33 31.5 mm to (124.7, 114.5), turned to 180 degrees
- moved R14 20.8 mm to (124.3, 117.0), turned to -90 degrees
- moved C15 20.6 mm to (131.8, 120.1), turned to 180 degrees
- moved C9 19.0 mm to (127.8, 114.5), turned to 0 degrees
- moved L1 15.3 mm to (132.7, 115.8)
- moved C10 14.9 mm to (122.8, 117.0), turned to -90 degrees
- moved C11 10.3 mm to (131.8, 122.5), turned to 180 degrees
- moved C7 5.05 mm to (127.1, 122.5)
Connections:
- C10 pad 1: Net-(U5-FB) -> Net-(U2-FB)
- C10 pad 2: +5V -> /Power+USB/BUCK_5V
- C11 pad 1: +5V -> /Power+USB/BUCK_5V
- C15 pad 1: +5V -> /Power+USB/BUCK_5V
- C5 pad 1: /ESP32+CH340/CH340_XO -> /Power+USB/VBUS_USBC
- C8 pad 1: +3V3 -> Net-(Q14-D)
- C9 pad 1: Net-(U5-BST) -> Net-(U2-BST)
- C9 pad 2: Net-(U5-SW) -> Net-(U2-SW)
- FB1 pad 1: +5V -> /Power+USB/VBUS_USBC
- FB1 pad 2: Net-(U6-EN) -> Net-(Q14-D)
- J1 pad A6: /Power+USB/D+ -> /Power+USB/USBC_P
- J1 pad A7: /Power+USB/D- -> /Power+USB/USBC_N
- J1 pad B6: /Power+USB/D+ -> /Power+USB/USBC_P
- J1 pad B7: /Power+USB/D- -> /Power+USB/USBC_N
- L1 pad 1: Net-(U5-SW) -> Net-(U2-SW)
- L1 pad 2: +5V -> /Power+USB/BUCK_5V
- Q14 pad 1: unconnected-(Q14-G-Pad1) -> /Power+USB/BUCK_5V
- Q14 pad 3: /Power+USB/VBUS_USBC -> Net-(Q14-D)
- Q5 pad 2: Net-(D1-K) -> /Power+USB/VLED
- R14 pad 1: Net-(U5-FB) -> Net-(U2-FB)
- R14 pad 2: +5V -> /Power+USB/BUCK_5V
- R3 pad 1: Net-(U1-TXD) -> Net-(U9-TXD)
- R33 pad 2: Net-(U5-FB) -> Net-(U2-FB)
- R4 pad 1: Net-(U1-RXD) -> Net-(U9-RXD)
- U1 pad 13: Net-(Q3-E) -> unconnected-(U1-IO14-Pad13)
- U1 pad 14: Net-(Q2-E) -> IR_CTRL
- U1 pad 15: unconnected-(U1-R232-Pad15) -> GND
- U1 pad 16: +3V3 -> unconnected-(U1-IO13-Pad16)
- U1 pad 2: Net-(U1-TXD) -> +3V3
- U1 pad 3: Net-(U1-RXD) -> EN
- U1 pad 4: +3V3 -> unconnected-(U1-SENSOR_VP-Pad4)
- U1 pad 5: USB_D+ -> unconnected-(U1-SENSOR_VN-Pad5)
- U1 pad 6: USB_D- -> V_SENSE
- U1 pad 7: /ESP32+CH340/CH340_XI -> unconnected-(U1-IO35-Pad7)
- U1 pad 8: /ESP32+CH340/CH340_XO -> unconnected-(U1-IO32-Pad8)
- U2 pad 1: /Power+USB/D- -> Net-(U2-FB)
- U2 pad 2: GND -> /Power+USB/BUCK_EN
- U2 pad 3: /Power+USB/D+ -> VIN
- U2 pad 4: USB_D+ -> GND
- U2 pad 5: /Power+USB/VBUS_USBC -> Net-(U2-SW)
- U2 pad 6: USB_D- -> Net-(U2-BST)
- U3 pad 1: GND -> /Power+USB/USBC_N
- U3 pad 2: +3V3 -> GND
- U3 pad 3: EN -> /Power+USB/USBC_P
- U3 pad 4: unconnected-(U3-SENSOR_VP-Pad4) -> /Power+USB/USB_D_P
- U3 pad 5: unconnected-(U3-SENSOR_VN-Pad5) -> /Power+USB/VBUS_USBC
- U3 pad 6: V_SENSE -> /Power+USB/USB_D_N
Other:
- board outline removed
