File: Hardware/1_ESP32_CH340.kicad_sch (KiCad schematic)
At the start: 64 parts, among them J4 Conn_01x04_Pin, J5 5mm Screw Terminal, J9 Conn_01x03_Pin, Q1 BC847, Q10 BC847, Q11 BC847, Q12 BC847, Q13 BC847, Q2 BC847, Q3 BC847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

Commit message: Update backups
Parts:
- removed C5: 30p, Capacitor_SMD:C_0603_1608Metric, symbol Device:C_Small
- removed C8: 10u, Diode_SMD:D_0805_2012Metric, symbol Device:C_Polarized_Small
- removed J9: Conn_01x03_Pin, Connector_PinHeader_2.54mm:PinHeader_1x03_P2.54mm_Vertical, symbol Connector:Conn_01x03_Pin
- removed U1: CH340G, Package_SO:SOIC-16_3.9x9.9mm_P1.27mm, symbol Interface_USB:CH340G
- removed U3: ESP32-WROOM-32D, RF_Module:ESP32-WROOM-32D, symbol RF_Module:ESP32-WROOM-32D
- removed Y1: 12MHz, Crystal:Crystal_SMD_3225-4Pin_3.2x2.5mm, symbol Device:Crystal_GND24
- added J6: Conn_01x03, symbol MG_Symbol_Lib:Conn_01x03
- added U1: ESP32-WROOM-32E, RF_Module:ESP32-WROOM-32D, symbol RF_Module:ESP32-WROOM-32E
- added U9: CH340C, Package_SO:SOIC-16_3.9x9.9mm_P1.27mm, symbol Interface_USB:CH340C
- C4: value 30p -> 10u; footprint Capacitor_SMD:C_0603_1608Metric -> (none)
Connections:
- net CH340_XI is gone; now on net +3V3: C4.1
- net +3V3: now also U1.2 (VDD), U9.16 (VCC), U9.4 (V3)
- net EN: now also U1.3 (EN)
- net ESP32_RX: now also J6.1 (Pin_1), U1.34 (RXD0/IO3)
- net ESP32_TX: now also J6.2 (Pin_2), U1.35 (TXD0/IO1)
- net GND: now also J6.3 (Pin_3), U1.1 (GND), U1.15 (GND), U1.38 (GND), U1.39 (GND), U9.1 (GND)
- net IO0: now also U1.25 (IO0)
- net IR_CTRL: now also U1.14 (IO12)
- net SCL: now also U1.36 (IO22)
- net SDA: now also U1.33 (IO21)
- net SW2: now also U1.26 (IO4)
- net SW3: now also U1.27 (IO16)
- net TEMP: now also U1.23 (IO15)
- net USB_D+: now also U9.5 (UD+)
- net USB_D-: now also U9.6 (UD-)
- net V_CTRL_BLUE: now also U1.30 (IO18)
- net V_CTRL_CW: now also U1.29 (IO5)
- net V_CTRL_GREEN: now also U1.31 (IO19)
- net V_CTRL_RED: now also U1.37 (IO23)
- net V_CTRL_WW: now also U1.28 (IO17)
- net V_SENSE: now also U1.6 (IO34)
- net at R3.1: now also U9.2 (TXD)
- net at Q2.2 (E), R7.1: now also U9.14 (~{RTS})
- net at Q3.2 (E), R6.1: now also U9.13 (~{DTR})
- net at R4.1: now also U9.3 (RXD)
- no-connect marks 19 -> 13
Other:
- note added: "IRLR8726 or AOD4184"
- note removed: "C_l = 2 * (C_load - C_stray)"
- note removed: "C_stray = 3-5 pF"
- note removed: "In case CH340C is used leave C1, C2, Y1 unpopulated"
- moved on the sheet: BOOT1, C14, D4, D5, D6, J4, Q7, R10, R11, R12, R13, R15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
