File: Hardware/2_power_usb.kicad_sch (KiCad schematic)
At the start: 25 parts, among them J1 USB_C_Receptacle_USB2.0, J3 Barrel_Jack_Switch, J7 5mm Screw Terminal, Q14 AO3401A, Q5 AOD4185, U2 USBLC6-2P6, U5 AP62300WU, U6 AP2112K-3.3, U8 LM321

Commit message: Update backups
Parts:
- removed FB1: 100R, Inductor_SMD:L_0603_1608Metric, symbol Device:FerriteBead
- removed U2: USBLC6-2P6, Package_TO_SOT_SMD:SOT-666, symbol Power_Protection:USBLC6-2P6
- removed U5: AP62300WU, Package_TO_SOT_SMD:TSOT-23-6, symbol Regulator_Switching:AP62300WU
- removed U8: LM321, Package_TO_SOT_SMD:SOT-23-5, symbol Amplifier_Operational:LM321
- added C17: 10u, Capacitor_SMD:C_1206_3216Metric, symbol MG_Symbol_Lib:CAP_1206
- added C5: 10n, Capacitor_SMD:C_0603_1608Metric, symbol MG_Symbol_Lib:CAP_0603
- added C8: 100n, Capacitor_SMD:C_0603_1608Metric, symbol MG_Symbol_Lib:CAP_0603
- added D2: SS34, Diode_SMD:D_SMA, symbol Diode:SS34
- added F2: 750mA, symbol Device:Fuse_Small
- added FB1: 100R 3A, Inductor_SMD:L_0603_1608Metric, symbol Device:FerriteBead_Small
- added J7: Conn_02x02_Odd_Even, symbol Connector_Generic:Conn_02x02_Odd_Even
- added R35: 10k, Resistor_SMD:R_0805_2012Metric, symbol Custom:R_0805
- added U2: AP63200WU, Package_TO_SOT_SMD:TSOT-23-6, symbol Regulator_Switching:AP63200WU
- added U3: USBLC6-2SC6, Package_TO_SOT_SMD:SOT-23-6, symbol Power_Protection:USBLC6-2SC6
- C11, C15: footprint Capacitor_SMD:C_0805_2012Metric -> Capacitor_SMD:C_1206_3216Metric
- C7: footprint Capacitor_SMD:C_0603_1608Metric -> Capacitor_SMD:C_1206_3216Metric
- renumbered J7 to J2, R5 to R14, R5 to R33
Connections:
- net +5V: now also D2.1 (K), F2.1, J7.2 (Pin_2); no longer C10.2, C11.1, C15.1, L1.2, R14.2
- net GND: now also C17.2, C5.2, C8.2, J7.4 (Pin_4), R35.2, U2.4 (GND), U3.2 (GND)
- net VBUS_USBC: now also C5.1, FB1.1, U3.5 (VBUS); no longer Q14.3 (D)
- net VIN: now also D1.1 (K), Q5.2 (S), J7.1 (Pin_1), U2.3 (IN)
- net at C10.1, R14.1, R33.2: now also U2.1 (FB)
- net at C9.2, L1.1: now also U2.5 (SW)
- net at C9.1: now also U2.6 (BST)
- net at C12.1, U6.1 (VIN), U6.3 (EN): now also F2.2
- net BUCK_5V: now reaches Q14.1 (G)
- net BUCK_5V: now also C10.2, C11.1, C15.1, L1.2, R14.2, D2.2 (A), R35.1
- net D+ renamed USBC_P
- net USBC_P: now also U3.3 (I/O2)
- net D- renamed USBC_N
- net USBC_N: now also U3.1 (I/O1)
- new net: C17.1, C8.1, FB1.2, Q14.3 (D)
- new net BUCK_EN: J7.3 (Pin_3), U2.2 (EN)
- new net USB_D_N: U3.6 (I/O1)
- new net USB_D_P: U3.4 (I/O2)
Other:
- moved on the sheet: C12, C13, C7, U6
